File: kicad-c128d/C128DCR Dual SID.kicad_pcb (KiCad board)
At the start: 2 copper layers, 67.8 x 41 mm, 21 parts, among them J4 ~{CS}, U1 MOS_6581, U2 MOS_6581

Commit message: plot values on silkscreen in generated gerber files
Other:
- board text added: "<- socket"
- board text added: "pins ->"
Changed lines of the file:
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@@
       (psa4output false)
       (plotreference true)
-      (plotvalue false)
+      (plotvalue true)
       (plotinvisibletext false)
       (sketchpadsonfab false)
@@
     (effects (font (size 0.8 0.8) (thickness 0.15)) (justify mirror))
   )
+  (gr_text "pins ->" (at 120.396 90.17) (layer "F.SilkS")
+    (effects (font (size 1 1) (thickness 0.15)) (justify right))
+  )
   (gr_text "Secondary\nSID" (at 158.496 106.0958 270) (layer "F.SilkS")
     (effects (font (size 1 1) (thickness 0.15)))
   )
+  (gr_text "<- socket" (at 127.254 90.17) (layer "F.SilkS")
+    (effects (font (size 1 1) (thickness 0.15)) (justify left))
+  )
   (gr_text "6581 C70/C71: 470pF (C128D default)\n8580 C70/C71: 22nF" (at 162.433 90.3732 270) (layer "F.SilkS")
